Commit message: attempt to solve stability issues
- making front camera mass-less
- lowering wheel damping
- modifying wheel Separation

File: Project2/catkin_ws/src/my_robot/urdf/scout_robot.xacro (robot description, xacro)
@@ -14,5 +14,5 @@
     <axis xyz="0 1 0" rpy="0 0 0"/>
     <limit effort="10000" velocity="1000"/>
-    <dynamics damping="1.0" friction="1.0"/>
+    <dynamics damping="0.5" friction="1.0"/>
   </joint>
   <joint type="continuous" name="back_left_wheel_hinge">
@@ -22,5 +22,5 @@
     <axis xyz="0 1 0" rpy="0 0 0"/>
     <limit effort="10000" velocity="1000"/>
-    <dynamics damping="1.0" friction="1.0"/>
+    <dynamics damping="0.5" friction="1.0"/>
   </joint>
   <joint type="continuous" name="front_right_wheel_hinge">
@@ -30,5 +30,5 @@
     <axis xyz="0 1 0" rpy="0 0 0"/>
     <limit effort="10000" velocity="1000"/>
-    <dynamics damping="1.0" friction="1.0"/>
+    <dynamics damping="0.5" friction="1.0"/>
   </joint>
   <joint type="continuous" name="back_right_wheel_hinge">
@@ -38,5 +38,5 @@
     <axis xyz="0 1 0" rpy="0 0 0"/>
     <limit effort="10000" velocity="1000"/>
-    <dynamics damping="1.0" friction="1.0"/>
+    <dynamics damping="0.5" friction="1.0"/>
   </joint>
   <joint type="fixed" name="camera_joint">
@@ -76,25 +76,25 @@
     </visual>
     <!-- <collision name='back_caster_collision'>
-      <origin xyz="-0.15 0 -0.05" rpy=" 0 0 0"/>
-      <geometry>
-        <sphere radius="0.0499"/>
-      </geometry>
-    </collision> -->
-    <!-- <visual name='back_caster_visual'>
-      <origin xyz="-0.15 0 -0.05" rpy=" 0 0 0"/>
-      <geometry>
-        <sphere radius="0.05"/>
-      </geometry>
-    </visual> -->
-    <!-- <collision name='front_caster_collision'>
-      <origin xyz="0.15 0 -0.05" rpy=" 0 0 0"/>
-      <geometry>
-        <sphere radius="0.0499"/>
+      <origin xyz="-0.035 0 -0.007" rpy=" 0 0 0"/>
+      <geometry>
+        <sphere radius="0.01399"/>
+      </geometry>
+    </collision>
+    <visual name='back_caster_visual'>
+      <origin xyz="-0.035 0 -0.007" rpy=" 0 0 0"/>
+      <geometry>
+        <sphere radius="0.014"/>
+      </geometry>
+    </visual>
+    <collision name='front_caster_collision'>
+      <origin xyz="0.045 0 -0.007" rpy=" 0 0 0"/>
+      <geometry>
+        <sphere radius="0.01399"/>
       </geometry>
     </collision>
     <visual name='front_caster_visual'>
-      <origin xyz="0.15 0 -0.05" rpy=" 0 0 0"/>
-      <geometry>
-        <sphere radius="0.05"/>
+      <origin xyz="0.045 0 -0.007" rpy=" 0 0 0"/>
+      <geometry>
+        <sphere radius="0.014"/>
       </geometry>
     </visual> -->
@@ -206,5 +206,5 @@
     </collision>
     <inertial>
-     <mass value="0.1"/>
+     <mass value="1e-5"/>
       <origin xyz="0 0 0" rpy="0 0 0" />
       <inertia

Commit message: configuring inertia matricies

File: Project2/catkin_ws/src/my_robot/urdf/scout_robot.xacro (robot description, xacro)
@@ -52,144 +52,78 @@
     <axis xyz="0 1 0" rpy="0 0 0"/>
   </joint>
-  <link name='chassis'>
-    <pose>0 0 0.1 0 0 0</pose>
-    <inertial>
-      <mass value="2.26797"/>
-      <origin xyz="0.0 0 0" rpy=" 0 0 0"/>
-      <inertia
-          ixx="0.1" ixy="0" ixz="0"
-          iyy="0.1" iyz="0"
-          izz="0.1"
-      />
-    </inertial>
-    <collision name='collision'>
-      <origin xyz="0 0 0.015" rpy=" 0 0 0"/>
-      <geometry>
-        <box size=".096 .047 .045"/>
-      </geometry>
-    </collision>
-    <visual name='chassis_visual'>
-      <origin xyz="0 0 0.015" rpy=" 0 0 0"/>
-      <geometry>
-        <box size=".096 .047 .045"/>
-      </geometry>
-    </visual>
-    <!-- <collision name='back_caster_collision'>
-      <origin xyz="-0.035 0 -0.007" rpy=" 0 0 0"/>
-      <geometry>
-        <sphere radius="0.01399"/>
-      </geometry>
-    </collision>
-    <visual name='back_caster_visual'>
-      <origin xyz="-0.035 0 -0.007" rpy=" 0 0 0"/>
-      <geometry>
-        <sphere radius="0.014"/>
-      </geometry>
-    </visual>
-    <collision name='front_caster_collision'>
-      <origin xyz="0.045 0 -0.007" rpy=" 0 0 0"/>
-      <geometry>
-        <sphere radius="0.01399"/>
-      </geometry>
-    </collision>
-    <visual name='front_caster_visual'>
-      <origin xyz="0.045 0 -0.007" rpy=" 0 0 0"/>
-      <geometry>
-        <sphere radius="0.014"/>
-      </geometry>
-    </visual> -->
+<!-- WHEEL MACRO
+    where radius and length are in meters
+    mass is in kg
+   -->
+  <xacro:macro
+    name="chassis"
+    params="name:=chassis x:=0.096 y:=0.047 height=0.045 mass:=0.26 off_the_ground:=0.015">
+    <link name='chassis'>
+      <inertial>
+        <mass value="${mass}"/>
+        <origin xyz="0 0 ${off_the_ground}" rpy=" 0 0 0"/>
+        <!-- INERTIA FORMULAS: https://en.wikipedia.org/wiki/List_of_moments_of_inertia -->
+        <inertia
+            ixx="${(1/12)*mass*((height*height)+(y*y))}" ixy="0" ixz="0"
+            iyy="${(1/12)*mass*((x*x)+(y*y))}" iyz="0"
+            izz="${(1/12)*mass*((x*x)+(height*height))}"
+        />
+      </inertial>
+      <collision name='${name}_collision'>
+        <origin xyz="0 0 ${off_the_ground}" rpy=" 0 0 0"/>
+        <geometry>
+          <box size="${x} ${y} ${height}"/>
+        </geometry>
+      </collision>
+      <visual name='${name}_visual'>
+        <origin xyz="0 0 ${off_the_ground}" rpy=" 0 0 0"/>
+        <geometry>
+          <box size="${x} ${y} ${height}"/>
+        </geometry>
+      </visual>
+    </link>
+  </xacro:macro>
+  <xacro:chassis />
+  <!-- WHEEL MACRO
+    where radius and length are in meters
+    mass is in kg
+   -->
+  <xacro:macro
+    name="wheel"
+    params="name radius:=0.02188 length:=0.025 mass:=0.025">
+  <link name="${name}">
+    <visual name="${name}_visual">
+        <origin xyz="0 0 0" rpy="0 1.57 1.57" />
+        <geometry>
+          <cylinder length="${length}" radius="${radius}" />
+        </geometry>
+      </visual>
+      <collision name="${name}_collision">
+        <origin xyz="0 0 0" rpy="0 1.57 1.57" />
+        <geometry>
+          <cylinder length="${length}" radius="${radius}" />
+        </geometry>
+      </collision>
+      <inertial>
+      <mass value="${mass}"/>
+        <origin xyz="0 0 0" rpy="0 1.57 1.57" />
+        <!-- INERTIA FORMULAS: https://en.wikipedia.org/wiki/List_of_moments_of_inertia -->
+        <!-- <inertia
+            ixx="${((1/12)*mass)*((3*(radius*radius)) + (length * length))}" ixy="0" ixz="0"
+            iyy="${((1/12)*mass)*((3*(radius*radius)) + (length * length))}" iyz="0"
+            izz="${(1/2)*mass*(radius*radius)}"
+        /> -->
+        <inertia
+            ixx="${((1/12)*mass)*((3*(radius*radius)) + (length * length))}" ixy="0" ixz="0"
+            iyy="${((1/12)*mass)*((3*(radius*radius)) + (length * length))}" iyz="0"
+            izz="${((1/12)*mass)*((3*(radius*radius)) + (length * length))}"
+        />
+      </inertial>
   </link>
-  <link name="front_left_wheel">
-    <visual name="front_left_wheel_visual">
-      <origin xyz="0 0 0" rpy="0 1.57 1.57" />
-      <geometry>
-        <cylinder length="0.025" radius="0.02188" />
-      </geometry>
-    </visual>
-    <collision name="front_left_wheel_collision">
-      <origin xyz="0 0 0" rpy="0 1.57 1.57" />
-      <geometry>
-        <cylinder length="0.025" radius="0.02188" />
-      </geometry>
-    </collision>
-    <inertial>
-     <mass value="0.75"/>
-      <origin xyz="0 0 0" rpy="0 1.57 1.57" />
-      <inertia
-          ixx="0.1" ixy="0" ixz="0"
-          iyy="0.1" iyz="0"
-          izz="0.1"
-      />
-    </inertial>
-  </link>
-  <link name="back_left_wheel">
-    <visual name="back_left_wheel_visual">
-      <origin xyz="0 0 0" rpy="0 1.57 1.57" />
-      <geometry>
-        <cylinder length="0.025" radius="0.02188" />
-      </geometry>
-    </visual>
-    <collision name="back_left_wheel_collision">
-      <origin xyz="0 0 0" rpy="0 1.57 1.57" />
-      <geometry>
-        <cylinder length="0.025" radius="0.02188" />
-      </geometry>
-    </collision>
-    <inertial>
-     <mass value="0.75"/>
-      <origin xyz="0 0 0" rpy="0 1.57 1.57" />
-      <inertia
-          ixx="0.1" ixy="0" ixz="0"
-          iyy="0.1" iyz="0"
-          izz="0.1"
-      />
-    </inertial>
-  </link>
-  <link name="front_right_wheel">
-    <visual name="front_right_wheel_visual">
-      <origin xyz="0 0 0" rpy="0 1.57 1.57" />
-      <geometry>
-        <cylinder length="0.025" radius="0.02188" />
-      </geometry>
-    </visual>
-    <collision name="front_right_wheel_collision">
-      <origin xyz="0 0 0" rpy="0 1.57 1.57" />
-      <geometry>
-        <cylinder length="0.025" radius="0.02188" />
-      </geometry>
-    </collision>
-    <inertial>
-     <mass value="0.75"/>
-      <origin xyz="0 0 0" rpy="0 1.57 1.57" />
-      <inertia
-          ixx="0.1" ixy="0" ixz="0"
-          iyy="0.1" iyz="0"
-          izz="0.1"
-      />
-    </inertial>
-  </link>
-  <link name="back_right_wheel">
-    <visual name="back_right_wheel_visual">
-      <origin xyz="0 0 0" rpy="0 1.57 1.57" />
-      <geometry>
-        <cylinder length="0.025" radius="0.02188" />
-      </geometry>
-    </visual>
-    <collision name="back_right_wheel_collision">
-      <origin xyz="0 0 0" rpy="0 1.57 1.57" />
-      <geometry>
-        <cylinder length="0.025" radius="0.02188" />
-      </geometry>
-    </collision>
-    <inertial>
-     <mass value="0.75"/>
-      <origin xyz="0 0 0" rpy="0 1.57 1.57" />
-      <inertia
-          ixx="0.1" ixy="0" ixz="0"
-          iyy="0.1" iyz="0"
-          izz="0.1"
-      />
-    </inertial>
-  </link>
+  </xacro:macro>
+  <xacro:wheel name="front_left_wheel"/>
+  <xacro:wheel name="back_left_wheel"/>
+  <xacro:wheel name="front_right_wheel"/>
+  <xacro:wheel name="back_right_wheel"/>
   <link name="camera">
     <visual name="camera_visual">

Commit message: working configs
- changing friction, damping, and torque

File: Project2/catkin_ws/src/my_robot/urdf/scout_robot.xacro (robot description, xacro)
@@ -8,36 +8,21 @@
     <child link="chassis" />
   </joint>
-  <joint type="continuous" name="front_left_wheel_hinge">
-    <origin xyz="0.02188 0.0365 0" rpy="0 0 0"/>
-    <child link="front_left_wheel"/>
-    <parent link="chassis"/>
-    <axis xyz="0 1 0" rpy="0 0 0"/>
-    <limit effort="10000" velocity="1000"/>
-    <dynamics damping="0.5" friction="1.0"/>
-  </joint>
-  <joint type="continuous" name="back_left_wheel_hinge">
-    <origin xyz="-0.03188 0.0365 0" rpy="0 0 0"/>
-    <child link="back_left_wheel"/>
-    <parent link="chassis"/>
-    <axis xyz="0 1 0" rpy="0 0 0"/>
-    <limit effort="10000" velocity="1000"/>
-    <dynamics damping="0.5" friction="1.0"/>
-  </joint>
-  <joint type="continuous" name="front_right_wheel_hinge">
-    <origin xyz="0.02188 -0.0365 0" rpy="0 0 0"/>
-    <child link="front_right_wheel"/>
-    <parent link="chassis"/>
-    <axis xyz="0 1 0" rpy="0 0 0"/>
-    <limit effort="10000" velocity="1000"/>
-    <dynamics damping="0.5" friction="1.0"/>
-  </joint>
-  <joint type="continuous" name="back_right_wheel_hinge">
-    <origin xyz="-0.03188 -0.0365 0" rpy="0 0 0"/>
-    <child link="back_right_wheel"/>
-    <parent link="chassis"/>
-    <axis xyz="0 1 0" rpy="0 0 0"/>
-    <limit effort="10000" velocity="1000"/>
-    <dynamics damping="0.5" friction="1.0"/>
-  </joint>
+  <!-- WHEEL JOINT MACRO -->
+  <xacro:macro
+    name="wheel_joint"
+    params="wheel_name ox oy">
+    <joint type="continuous" name="${wheel_name}_hinge">
+      <origin xyz="${ox} ${oy} 0" rpy="0 0 0"/>
+      <child link="${wheel_name}"/>
+      <parent link="chassis"/>
+      <axis xyz="0 1 0" rpy="0 0 0"/>
+      <limit effort="1000" velocity="1000"/>
+      <dynamics damping="1e-6" friction="1e-6"/>
+    </joint>
+  </xacro:macro>
+  <xacro:wheel_joint wheel_name="front_left_wheel" ox="0.02188" oy="0.0365" />
+  <xacro:wheel_joint wheel_name="back_left_wheel" ox="-0.03188" oy="0.0365" />
+  <xacro:wheel_joint wheel_name="front_right_wheel" ox="0.02188" oy="-0.0365" />
+  <xacro:wheel_joint wheel_name="back_right_wheel" ox="-0.03188" oy="-0.0365" />
   <joint type="fixed" name="camera_joint">
     <origin xyz="0.055 0 0.015" rpy="0 0 0"/>
@@ -93,5 +78,5 @@
     params="name radius:=0.02188 length:=0.025 mass:=0.025">
   <link name="${name}">
-    <visual name="${name}_visual">
+      <visual name="${name}_visual">
         <origin xyz="0 0 0" rpy="0 1.57 1.57" />
         <geometry>
@@ -105,14 +90,14 @@
         </geometry>
       </collision>
-      <inertial>
-      <mass value="${mass}"/>
-        <origin xyz="0 0 0" rpy="0 1.57 1.57" />
-        <!-- INERTIA FORMULAS: https://en.wikipedia.org/wiki/List_of_moments_of_inertia -->
-        <!-- This commented out formula is the one wikipedia suggests, but by using the izz, it doesn't look good in gazebo -->
-        <!-- <inertia
+      <!-- INERTIA FORMULAS: https://en.wikipedia.org/wiki/List_of_moments_of_inertia -->
+      <!-- This commented out formula is the one wikipedia suggests, but by using the izz, it doesn't look good in gazebo -->
+      <!-- <inertia
             ixx="${((1/12)*mass)*((3*(radius*radius)) + (length * length))}" ixy="0" ixz="0"
             iyy="${((1/12)*mass)*((3*(radius*radius)) + (length * length))}" iyz="0"
             izz="${(1/2)*mass*(radius*radius)}"
         /> -->
+      <inertial>
+        <mass value="${mass}"/>
+        <origin xyz="0 0 0" rpy="0 1.57 1.57" />
         <inertia
             ixx="${((1/12)*mass)*((3*(radius*radius)) + (length * length))}" ixy="0" ixz="0"
